Commit message: switched to pose publisher for absolute coord

File: urdf/diff_robot.urdf (robot description, URDF)
Before this commit: robot diff_robot, 5 links, 4 joints
Links:
- added link skid_plate_front, mass 0.18; collision box size=0.15 0.18 0.015; visual box size=0.15 0.18 0.015
Joints:
- added joint skid_joint_front: type fixed, parent base_link, child skid_plate_front, origin xyz=0.27 0 -0.1725 rpy=0 0 0
- joint skid_joint: origin xyz=-0.27 0 -0.135 rpy=0 0 0 -> xyz=-0.27 0 -0.1725 rpy=0 0 0

Commit message: Fixed bugs

File: urdf/diff_robot.urdf (robot description, URDF)
Before this commit: robot diff_robot, 6 links, 5 joints
Links:
- added link accent_ring, mass 0.05; collision cylinder length=0.001 radius=0.001; visual cylinder length=0.018 radius=0.37
- added link dome_lens, mass 0.01; collision cylinder length=0.001 radius=0.001; visual cylinder length=0.008 radius=0.035
- added link left_rim, mass 0.05; collision box size=0.001 0.001 0.001; visual cylinder length=0.080 radius=0.085
- added link right_rim, mass 0.05; collision box size=0.001 0.001 0.001; visual cylinder length=0.080 radius=0.085
- added link sensor_dome, mass 0.25; collision cylinder length=0.05 radius=0.09; visual cylinder length=0.05 radius=0.09
- added link top_plate, mass 0.2; collision cylinder length=0.001 radius=0.001; visual cylinder length=0.012 radius=0.34
Joints:
- added joint accent_ring_joint: type fixed, parent base_link, child accent_ring, origin xyz=0 0 0.01 rpy=0 0 0
- added joint dome_lens_joint: type fixed, parent sensor_dome, child dome_lens, origin xyz=0 0 0.029 rpy=0 0 0
- added joint left_rim_joint: type fixed, parent left_wheel, child left_rim, origin xyz=0 0 0 rpy=0 0 0
- added joint right_rim_joint: type fixed, parent right_wheel, child right_rim, origin xyz=0 0 0 rpy=0 0 0
- added joint sensor_dome_joint: type fixed, parent base_link, child sensor_dome, origin xyz=0.08 0 0.055 rpy=0 0 0
- added joint top_plate_joint: type fixed, parent base_link, child top_plate, origin xyz=0 0 0.036 rpy=0 0 0
